Commit message: rabbit check

File: urdf/common/imu.urdf.xacro (robot description, xacro)
@@ -33,7 +33,7 @@
         <xacro:if value="$(arg use_sim)">
             <gazebo>
-                <plugin name="rm_ros_control" filename="librm_robot_hw_sim.so">
+                <plugin name="rc_ros_control" filename="librc_robot_hw_sim.so">
                     <robotNamespace>/</robotNamespace>
-                    <robotSimType>rm_gazebo/RmRobotHWSim</robotSimType>
+                    <robotSimType>rc_gazebo/RmRobotHWSim</robotSimType>
                 </plugin>
             </gazebo>

File: urdf/common/radar.urdf.xacro (robot description, xacro)
@@ -47,7 +47,7 @@
                                 <samples>360</samples>
                                 <resolution>1</resolution>
-                                <min_angle>0.0</min_angle>
+                                <min_angle>-1.5707963</min_angle>
                                 <!--                        <max_angle>6.1</max_angle>-->
-                                <max_angle>6.28319</max_angle>
+                                <max_angle>1.5707963</max_angle>
                             </horizontal>
                         </scan>

File: urdf/engineer/chassis.urdf.xacro (robot description, xacro)
@@ -1,4 +1,4 @@
 <robot xmlns:xacro="http://www.ros.org/wiki/xacro" name="chassis">
-    <xacro:include filename="$(find rm_description)/urdf/common/swerve_drive.urdf.xacro"/>
+    <xacro:include filename="$(find rc_description)/urdf/common/swerve_drive.urdf.xacro"/>
     <!-- https://upload.wikimedia.org/wikipedia/commons/5/52/Wheelbase_and_Track.png -->
     <xacro:property name="wheel_track" value="0.423"/>
@@ -6,4 +6,6 @@
     <xacro:property name="wheel_offset_z" value="0.06795"/>
     <xacro:macro name="chassis">
+        <link name="dummy">
+        </link>
         <link name="base_link">
             <inertial>
@@ -115,4 +117,8 @@
             </collision>
         </link>
+        <joint name="dummy_joint" type="fixed">
+            <parent link="dummy"/>
+            <child link="base_link"/>
+        </joint>
         <!--        <link name="card">-->
         <!--            <inertial>-->

File: urdf/engineer/engineer.urdf.xacro (robot description, xacro)
@@ -5,6 +5,7 @@
     <xacro:arg name="load_radar" default="true"/>
     <xacro:arg name="load_action" default="true"/>
-    <xacro:arg name="load_arm" default="false"/>
-    <xacro:arg name="use_sim" default="false"/>
+    <xacro:arg name="load_arm" default="true"/>
+    <xacro:arg name="use_sim" default="true"/>
+    <xacro:arg name="use_simulation" default="false"/>
     <xacro:if value="$(arg load_chassis)">
         <xacro:include filename="$(find rc_description)/urdf/engineer/chassis.urdf.xacro"/>
@@ -23,19 +24,19 @@
                       rpy="0.0 0.0 0.0"/>
     </xacro:if>
-    <!--    <xacro:if value="$(arg use_sim)">-->
-    <!--        <gazebo>-->
-    <!--            <plugin name="gazebo_ros_control" filename="libgazebo_ros_control.so">-->
-    <!--                <robotNamespace>/</robotNamespace>-->
-    <!--            </plugin>-->
-    <!--        </gazebo>-->
-    <!--    </xacro:if>-->
-    <!--    <xacro:if value="$(arg use_sim)">-->
-    <!--        <gazebo>-->
-    <!--            <plugin name="rm_ros_control" filename="librm_robot_hw_sim.so">-->
-    <!--                <robotNamespace>/</robotNamespace>-->
-    <!--                <robotSimType>rm_gazebo/RmRobotHWSim</robotSimType>-->
-    <!--            </plugin>-->
-    <!--        </gazebo>-->
-    <!--    </xacro:if>-->
+       <!-- <xacro:if value="$(arg use_sim)">
+           <gazebo>
+                <plugin name="gazebo_ros_control" filename="libgazebo_ros_control.so">
+                    <robotNamespace>/</robotNamespace>
+               </plugin>
+           </gazebo>
+       </xacro:if> -->
+    <!-- <xacro:if value="$(arg use_sim)">
+        <gazebo>
+            <plugin name="rc_ros_control" filename="librm_robot_hw_sim.so">
+                <robotNamespace>/</robotNamespace>
+                <robotSimType>rc_gazebo/RmRobotHWSim</robotSimType>
+            </plugin>
+        </gazebo>
+    </xacro:if> -->
     <xacro:if value="$(arg load_arm)">
         <xacro:include filename="$(find rc_description)/urdf/engineer/arm.urdf.xacro"/>

File: urdf/standard/chassis.urdf.xacro (robot description, xacro)
@@ -1,4 +1,4 @@
 <robot xmlns:xacro="http://www.ros.org/wiki/xacro">
-    <xacro:include filename="$(find rm_description)/urdf/common/omni_wheel.urdf.xacro"/>
+    <xacro:include filename="$(find rc_description)/urdf/common/omni_wheel.urdf.xacro"/>
     <!-- https://upload.wikimedia.org/wikipedia/commons/5/52/Wheelbase_and_Track.png -->
     <xacro:property name="chassis_radius" value="0.196"/>
@@ -15,5 +15,5 @@
                 <origin xyz="0 0 0" rpy="0 0 0"/>
                 <geometry>
-                    <mesh filename="package://rm_description/meshes/standard/base.stl" scale="0.001 0.001 0.001"/>
+                    <mesh filename="package://rc_description/meshes/standard/base.stl" scale="0.001 0.001 0.001"/>
                 </geometry>
             </visual>

File: urdf/standard/gimbal.urdf.xacro (robot description, xacro)
@@ -14,5 +14,5 @@
             <origin xyz="0 0 0" rpy="0 0 0"/>
             <geometry>
-                <mesh filename="package://rm_description/meshes/standard/yaw.stl" scale="0.001 0.001 0.001"/>
+                <mesh filename="package://rc_description/meshes/standard/yaw.stl" scale="0.001 0.001 0.001"/>
             </geometry>
         </visual>
@@ -20,5 +20,5 @@
             <origin xyz="0 0 0" rpy="0 0 0"/>
             <geometry>
-                <mesh filename="package://rm_description/meshes/standard/yaw.stl" scale="0.001 0.001 0.001"/>
+                <mesh filename="package://rc_description/meshes/standard/yaw.stl" scale="0.001 0.001 0.001"/>
             </geometry>
         </collision>
@@ -49,5 +49,5 @@
             <origin xyz="0 0 0" rpy="0 0 0"/>
             <geometry>
-                <mesh filename="package://rm_description/meshes/standard/pitch.stl" scale="0.001 0.001 0.001"/>
+                <mesh filename="package://rc_description/meshes/standard/pitch.stl" scale="0.001 0.001 0.001"/>
             </geometry>
         </visual>
@@ -55,5 +55,5 @@
             <origin xyz="0 0 0" rpy="0 0 0"/>
             <geometry>
-                <mesh filename="package://rm_description/meshes/standard/pitch.stl" scale="0.001 0.001 0.001"/>
+                <mesh filename="package://rc_description/meshes/standard/pitch.stl" scale="0.001 0.001 0.001"/>
             </geometry>
         </collision>

File: urdf/standard/shooter.urdf.xacro (robot description, xacro)
@@ -1,5 +1,5 @@
 <robot xmlns:xacro="http://www.ros.org/wiki/xacro">
-    <xacro:include filename="$(find rm_description)/urdf/common/friction.urdf.xacro"/>
-    <!--    <xacro:include filename="$(find rm_description)/urdf/standard/gimbal.urdf.xacro"/>-->
+    <xacro:include filename="$(find rc_description)/urdf/common/friction.urdf.xacro"/>
+    <!--    <xacro:include filename="$(find rc_description)/urdf/standard/gimbal.urdf.xacro"/>-->
     <xacro:property name="wheel_offset_x" value="0.047"/>
     <xacro:property name="wheel_offset_y" value="0.0365"/>
@@ -21,5 +21,5 @@
             <origin xyz="0 0 0" rpy="0 0 0"/>
             <geometry>
-                <mesh filename="package://rm_description/meshes/standard/trigger.stl" scale="0.001 0.001 0.001"/>
+                <mesh filename="package://rc_description/meshes/standard/trigger.stl" scale="0.001 0.001 0.001"/>
             </geometry>
         </visual>
@@ -27,5 +27,5 @@
             <origin xyz="0 0 0" rpy="0 0 0"/>
             <geometry>
-                <mesh filename="package://rm_description/meshes/standard/trigger.stl" scale="0.001 0.001 0.001"/>
+                <mesh filename="package://rc_description/meshes/standard/trigger.stl" scale="0.001 0.001 0.001"/>
             </geometry>
         </collision>

File: urdf/standard/standard.urdf.xacro (robot description, xacro)
@@ -1,7 +1,7 @@
 <?xml version="1.0"?>
 <robot xmlns:xacro="http://www.ros.org/wiki/xacro" name="standard3">
-    <!--    ref:https://github.com/rm-controls-->
+    <!--    ref:https://github.com/rc-controls-->
     <xacro:arg name="load_chassis" default="true"/>
-    <xacro:arg name="load_gimbal" default="true"/>
+    <xacro:arg name="load_gimbal" default="false"/>
     <xacro:arg name="load_shooter" default="true"/>
     <xacro:arg name="camera_link" default="camera_link"/>
@@ -11,11 +11,11 @@
     <xacro:arg name="roller_type" default="realistic"/>
     <xacro:if value="$(arg load_chassis)">
-        <xacro:include filename="$(find rm_description)/urdf/standard/chassis.urdf.xacro"/>
+        <xacro:include filename="$(find rc_description)/urdf/standard/chassis.urdf.xacro"/>
         <xacro:chassis roller_type="$(arg roller_type)"/>
         <xacro:if value="$(arg load_gimbal)">
-            <xacro:include filename="$(find rm_description)/urdf/standard/gimbal.urdf.xacro"/>
-            <xacro:include filename="$(find rm_description)/urdf/standard3/gimbal.transmission.urdf.xacro"/>
-            <xacro:include filename="$(find rm_description)/urdf/common/camera.urdf.xacro"/>
-            <xacro:include filename="$(find rm_description)/urdf/common/imu.urdf.xacro"/>
+            <xacro:include filename="$(find rc_description)/urdf/standard/gimbal.urdf.xacro"/>
+            <xacro:include filename="$(find rc_description)/urdf/standard3/gimbal.transmission.urdf.xacro"/>
+            <xacro:include filename="$(find rc_description)/urdf/common/camera.urdf.xacro"/>
+            <xacro:include filename="$(find rc_description)/urdf/common/imu.urdf.xacro"/>
             <xacro:camera_sensor xyz="0 0 0.0887" rpy="0 0 0" frame_id="$(arg camera_link)" parent="pitch"
                                  camera_sim="$(arg use_simulation)"/>
@@ -29,6 +29,6 @@
                        rpy="1.5487827 -0.0054278 -0.01"/>
             <xacro:if value="$(arg load_shooter)">
-                <xacro:include filename="$(find rm_description)/urdf/standard/shooter.urdf.xacro"/>
-                <xacro:include filename="$(find rm_description)/urdf/standard3/shooter.transmission.urdf.xacro"/>
+                <xacro:include filename="$(find rc_description)/urdf/standard/shooter.urdf.xacro"/>
+                <xacro:include filename="$(find rc_description)/urdf/standard3/shooter.transmission.urdf.xacro"/>
             </xacro:if>
         </xacro:if>
@@ -36,7 +36,7 @@
     <xacro:if value="$(arg use_simulation)">
         <gazebo>
-            <plugin name="rm_ros_control" filename="librm_robot_hw_sim.so">
+            <plugin name="rc_ros_control" filename="librc_robot_hw_sim.so">
                 <robotNamespace>/</robotNamespace>
-                <robotSimType>rm_gazebo/RmRobotHWSim</robotSimType>
+                <robotSimType>rc_gazebo/rcRobotHWSim</robotSimType>
             </plugin>
         </gazebo>

Commit message: Revert "rabbit check"
This reverts commit 7c36216bb156bbf7f551dc9beabc517aadc10322.

File: urdf/common/imu.urdf.xacro (robot description, xacro)
@@ -33,7 +33,7 @@
         <xacro:if value="$(arg use_sim)">
             <gazebo>
-                <plugin name="rc_ros_control" filename="librc_robot_hw_sim.so">
+                <plugin name="rm_ros_control" filename="librm_robot_hw_sim.so">
                     <robotNamespace>/</robotNamespace>
-                    <robotSimType>rc_gazebo/RmRobotHWSim</robotSimType>
+                    <robotSimType>rm_gazebo/RmRobotHWSim</robotSimType>
                 </plugin>
             </gazebo>

File: urdf/common/radar.urdf.xacro (robot description, xacro)
@@ -47,7 +47,7 @@
                                 <samples>360</samples>
                                 <resolution>1</resolution>
-                                <min_angle>-1.5707963</min_angle>
+                                <min_angle>0.0</min_angle>
                                 <!--                        <max_angle>6.1</max_angle>-->
-                                <max_angle>1.5707963</max_angle>
+                                <max_angle>6.28319</max_angle>
                             </horizontal>
                         </scan>

File: urdf/engineer/chassis.urdf.xacro (robot description, xacro)
@@ -1,4 +1,4 @@
 <robot xmlns:xacro="http://www.ros.org/wiki/xacro" name="chassis">
-    <xacro:include filename="$(find rc_description)/urdf/common/swerve_drive.urdf.xacro"/>
+    <xacro:include filename="$(find rm_description)/urdf/common/swerve_drive.urdf.xacro"/>
     <!-- https://upload.wikimedia.org/wikipedia/commons/5/52/Wheelbase_and_Track.png -->
     <xacro:property name="wheel_track" value="0.423"/>
@@ -6,6 +6,4 @@
     <xacro:property name="wheel_offset_z" value="0.06795"/>
     <xacro:macro name="chassis">
-        <link name="dummy">
-        </link>
         <link name="base_link">
             <inertial>
@@ -117,8 +115,4 @@
             </collision>
         </link>
-        <joint name="dummy_joint" type="fixed">
-            <parent link="dummy"/>
-            <child link="base_link"/>
-        </joint>
         <!--        <link name="card">-->
         <!--            <inertial>-->

File: urdf/engineer/engineer.urdf.xacro (robot description, xacro)
@@ -5,7 +5,6 @@
     <xacro:arg name="load_radar" default="true"/>
     <xacro:arg name="load_action" default="true"/>
-    <xacro:arg name="load_arm" default="true"/>
-    <xacro:arg name="use_sim" default="true"/>
-    <xacro:arg name="use_simulation" default="false"/>
+    <xacro:arg name="load_arm" default="false"/>
+    <xacro:arg name="use_sim" default="false"/>
     <xacro:if value="$(arg load_chassis)">
         <xacro:include filename="$(find rc_description)/urdf/engineer/chassis.urdf.xacro"/>
@@ -24,19 +23,19 @@
                       rpy="0.0 0.0 0.0"/>
     </xacro:if>
-       <!-- <xacro:if value="$(arg use_sim)">
-           <gazebo>
-                <plugin name="gazebo_ros_control" filename="libgazebo_ros_control.so">
-                    <robotNamespace>/</robotNamespace>
-               </plugin>
-           </gazebo>
-       </xacro:if> -->
-    <!-- <xacro:if value="$(arg use_sim)">
-        <gazebo>
-            <plugin name="rc_ros_control" filename="librm_robot_hw_sim.so">
-                <robotNamespace>/</robotNamespace>
-                <robotSimType>rc_gazebo/RmRobotHWSim</robotSimType>
-            </plugin>
-        </gazebo>
-    </xacro:if> -->
+    <!--    <xacro:if value="$(arg use_sim)">-->
+    <!--        <gazebo>-->
+    <!--            <plugin name="gazebo_ros_control" filename="libgazebo_ros_control.so">-->
+    <!--                <robotNamespace>/</robotNamespace>-->
+    <!--            </plugin>-->
+    <!--        </gazebo>-->
+    <!--    </xacro:if>-->
+    <!--    <xacro:if value="$(arg use_sim)">-->
+    <!--        <gazebo>-->
+    <!--            <plugin name="rm_ros_control" filename="librm_robot_hw_sim.so">-->
+    <!--                <robotNamespace>/</robotNamespace>-->
+    <!--                <robotSimType>rm_gazebo/RmRobotHWSim</robotSimType>-->
+    <!--            </plugin>-->
+    <!--        </gazebo>-->
+    <!--    </xacro:if>-->
     <xacro:if value="$(arg load_arm)">
         <xacro:include filename="$(find rc_description)/urdf/engineer/arm.urdf.xacro"/>

File: urdf/standard/chassis.urdf.xacro (robot description, xacro)
@@ -1,4 +1,4 @@
 <robot xmlns:xacro="http://www.ros.org/wiki/xacro">
-    <xacro:include filename="$(find rc_description)/urdf/common/omni_wheel.urdf.xacro"/>
+    <xacro:include filename="$(find rm_description)/urdf/common/omni_wheel.urdf.xacro"/>
     <!-- https://upload.wikimedia.org/wikipedia/commons/5/52/Wheelbase_and_Track.png -->
     <xacro:property name="chassis_radius" value="0.196"/>
@@ -15,5 +15,5 @@
                 <origin xyz="0 0 0" rpy="0 0 0"/>
                 <geometry>
-                    <mesh filename="package://rc_description/meshes/standard/base.stl" scale="0.001 0.001 0.001"/>
+                    <mesh filename="package://rm_description/meshes/standard/base.stl" scale="0.001 0.001 0.001"/>
                 </geometry>
             </visual>

File: urdf/standard/gimbal.urdf.xacro (robot description, xacro)
@@ -14,5 +14,5 @@
             <origin xyz="0 0 0" rpy="0 0 0"/>
             <geometry>
-                <mesh filename="package://rc_description/meshes/standard/yaw.stl" scale="0.001 0.001 0.001"/>
+                <mesh filename="package://rm_description/meshes/standard/yaw.stl" scale="0.001 0.001 0.001"/>
             </geometry>
         </visual>
@@ -20,5 +20,5 @@
             <origin xyz="0 0 0" rpy="0 0 0"/>
             <geometry>
-                <mesh filename="package://rc_description/meshes/standard/yaw.stl" scale="0.001 0.001 0.001"/>
+                <mesh filename="package://rm_description/meshes/standard/yaw.stl" scale="0.001 0.001 0.001"/>
             </geometry>
         </collision>
@@ -49,5 +49,5 @@
             <origin xyz="0 0 0" rpy="0 0 0"/>
             <geometry>
-                <mesh filename="package://rc_description/meshes/standard/pitch.stl" scale="0.001 0.001 0.001"/>
+                <mesh filename="package://rm_description/meshes/standard/pitch.stl" scale="0.001 0.001 0.001"/>
             </geometry>
         </visual>
@@ -55,5 +55,5 @@
             <origin xyz="0 0 0" rpy="0 0 0"/>
             <geometry>
-                <mesh filename="package://rc_description/meshes/standard/pitch.stl" scale="0.001 0.001 0.001"/>
+                <mesh filename="package://rm_description/meshes/standard/pitch.stl" scale="0.001 0.001 0.001"/>
             </geometry>
         </collision>

File: urdf/standard/shooter.urdf.xacro (robot description, xacro)
@@ -1,5 +1,5 @@
 <robot xmlns:xacro="http://www.ros.org/wiki/xacro">
-    <xacro:include filename="$(find rc_description)/urdf/common/friction.urdf.xacro"/>
-    <!--    <xacro:include filename="$(find rc_description)/urdf/standard/gimbal.urdf.xacro"/>-->
+    <xacro:include filename="$(find rm_description)/urdf/common/friction.urdf.xacro"/>
+    <!--    <xacro:include filename="$(find rm_description)/urdf/standard/gimbal.urdf.xacro"/>-->
     <xacro:property name="wheel_offset_x" value="0.047"/>
     <xacro:property name="wheel_offset_y" value="0.0365"/>
@@ -21,5 +21,5 @@
             <origin xyz="0 0 0" rpy="0 0 0"/>
             <geometry>
-                <mesh filename="package://rc_description/meshes/standard/trigger.stl" scale="0.001 0.001 0.001"/>
+                <mesh filename="package://rm_description/meshes/standard/trigger.stl" scale="0.001 0.001 0.001"/>
             </geometry>
         </visual>
@@ -27,5 +27,5 @@
             <origin xyz="0 0 0" rpy="0 0 0"/>
             <geometry>
-                <mesh filename="package://rc_description/meshes/standard/trigger.stl" scale="0.001 0.001 0.001"/>
+                <mesh filename="package://rm_description/meshes/standard/trigger.stl" scale="0.001 0.001 0.001"/>
             </geometry>
         </collision>

File: urdf/standard/standard.urdf.xacro (robot description, xacro)
@@ -1,7 +1,7 @@
 <?xml version="1.0"?>
 <robot xmlns:xacro="http://www.ros.org/wiki/xacro" name="standard3">
-    <!--    ref:https://github.com/rc-controls-->
+    <!--    ref:https://github.com/rm-controls-->
     <xacro:arg name="load_chassis" default="true"/>
-    <xacro:arg name="load_gimbal" default="false"/>
+    <xacro:arg name="load_gimbal" default="true"/>
     <xacro:arg name="load_shooter" default="true"/>
     <xacro:arg name="camera_link" default="camera_link"/>
@@ -11,11 +11,11 @@
     <xacro:arg name="roller_type" default="realistic"/>
     <xacro:if value="$(arg load_chassis)">
-        <xacro:include filename="$(find rc_description)/urdf/standard/chassis.urdf.xacro"/>
+        <xacro:include filename="$(find rm_description)/urdf/standard/chassis.urdf.xacro"/>
         <xacro:chassis roller_type="$(arg roller_type)"/>
         <xacro:if value="$(arg load_gimbal)">
-            <xacro:include filename="$(find rc_description)/urdf/standard/gimbal.urdf.xacro"/>
-            <xacro:include filename="$(find rc_description)/urdf/standard3/gimbal.transmission.urdf.xacro"/>
-            <xacro:include filename="$(find rc_description)/urdf/common/camera.urdf.xacro"/>
-            <xacro:include filename="$(find rc_description)/urdf/common/imu.urdf.xacro"/>
+            <xacro:include filename="$(find rm_description)/urdf/standard/gimbal.urdf.xacro"/>
+            <xacro:include filename="$(find rm_description)/urdf/standard3/gimbal.transmission.urdf.xacro"/>
+            <xacro:include filename="$(find rm_description)/urdf/common/camera.urdf.xacro"/>
+            <xacro:include filename="$(find rm_description)/urdf/common/imu.urdf.xacro"/>
             <xacro:camera_sensor xyz="0 0 0.0887" rpy="0 0 0" frame_id="$(arg camera_link)" parent="pitch"
                                  camera_sim="$(arg use_simulation)"/>
@@ -29,6 +29,6 @@
                        rpy="1.5487827 -0.0054278 -0.01"/>
             <xacro:if value="$(arg load_shooter)">
-                <xacro:include filename="$(find rc_description)/urdf/standard/shooter.urdf.xacro"/>
-                <xacro:include filename="$(find rc_description)/urdf/standard3/shooter.transmission.urdf.xacro"/>
+                <xacro:include filename="$(find rm_description)/urdf/standard/shooter.urdf.xacro"/>
+                <xacro:include filename="$(find rm_description)/urdf/standard3/shooter.transmission.urdf.xacro"/>
             </xacro:if>
         </xacro:if>
@@ -36,7 +36,7 @@
     <xacro:if value="$(arg use_simulation)">
         <gazebo>
-            <plugin name="rc_ros_control" filename="librc_robot_hw_sim.so">
+            <plugin name="rm_ros_control" filename="librm_robot_hw_sim.so">
                 <robotNamespace>/</robotNamespace>
-                <robotSimType>rc_gazebo/rcRobotHWSim</robotSimType>
+                <robotSimType>rm_gazebo/RmRobotHWSim</robotSimType>
             </plugin>
         </gazebo>
