Commit message: rabbit check

File: urdf/rabbit/chassis.urdf.xacro (robot description, xacro)
@@ -2,5 +2,5 @@
     <xacro:include filename="$(find rc_description)/urdf/common/mecanum_wheel.urdf.xacro"/>
     <xacro:property name="wheel_track" value="0.37116"/>
-    <xacro:property name="wheel_base" value="0.4164"/>
+    <xacro:property name="wheel_base" value="0.4664"/>
     <xacro:property name="wheel_offset_z" value="-0.02"/>
     <xacro:macro name="chassis" params="roller_type">
@@ -8,5 +8,5 @@
         </link>
         <link name="base_link">
-        <inertial>
+        <!-- <inertial>
         <origin
             xyz="0.0 7.68E-18 0.0122"
@@ -33,5 +33,29 @@
                         <mesh filename="package://rc_description/meshes/rabbit/base_link.stl" />
                     </geometry>
-                </collision>
+                </collision> -->
+        <!--test-->
+        <visual>
+            <geometry>
+                <cylinder radius="0.1" length="0.08" />
+            </geometry>
+            <origin xyz="0 0 0" rpy="0 0 0" />
+            <material name="yellow">
+                <color rgba="0.8 0.3 0.1 0.5" />
+            </material>
+        </visual>
+        <inertial>
+        <origin
+            xyz="0.0 0.0 0.0"
+            rpy="0 0 0" />
+        <mass
+            value="15" />
+        <inertia
+            ixx="0.0"
+            ixy="0.0"
+            ixz="0.0"
+            iyy="0.0"
+            iyz="0.0"
+            izz="0.0" />
+        </inertial>
         </link>
         <joint name="dummy_joint" type="fixed">

File: urdf/rabbit/rabbit.urdf.xacro (robot description, xacro)
@@ -47,11 +47,3 @@
                       rpy="0.0 0.0 0.0"/>
     </xacro:if>
-    <xacro:if value="$(arg use_simulation)">
-        <gazebo>
-            <plugin name="rc_ros_control" filename="librc_robot_hw_sim.so">
-                <robotNamespace>/</robotNamespace>
-                <robotSimType>rc_gazebo/rcRobotHWSim</robotSimType>
-            </plugin>
-        </gazebo>
-    </xacro:if>
 </robot>

Commit message: Revert "rabbit check"
This reverts commit 67a580101ec5a99e6cab7d9f5bef9a0c2d1b75f5.

File: urdf/rabbit/chassis.urdf.xacro (robot description, xacro)
@@ -2,5 +2,5 @@
     <xacro:include filename="$(find rc_description)/urdf/common/mecanum_wheel.urdf.xacro"/>
     <xacro:property name="wheel_track" value="0.37116"/>
-    <xacro:property name="wheel_base" value="0.4664"/>
+    <xacro:property name="wheel_base" value="0.4164"/>
     <xacro:property name="wheel_offset_z" value="-0.02"/>
     <xacro:macro name="chassis" params="roller_type">
@@ -8,5 +8,5 @@
         </link>
         <link name="base_link">
-        <!-- <inertial>
+        <inertial>
         <origin
             xyz="0.0 7.68E-18 0.0122"
@@ -33,29 +33,5 @@
                         <mesh filename="package://rc_description/meshes/rabbit/base_link.stl" />
                     </geometry>
-                </collision> -->
-        <!--test-->
-        <visual>
-            <geometry>
-                <cylinder radius="0.1" length="0.08" />
-            </geometry>
-            <origin xyz="0 0 0" rpy="0 0 0" />
-            <material name="yellow">
-                <color rgba="0.8 0.3 0.1 0.5" />
-            </material>
-        </visual>
-        <inertial>
-        <origin
-            xyz="0.0 0.0 0.0"
-            rpy="0 0 0" />
-        <mass
-            value="15" />
-        <inertia
-            ixx="0.0"
-            ixy="0.0"
-            ixz="0.0"
-            iyy="0.0"
-            iyz="0.0"
-            izz="0.0" />
-        </inertial>
+                </collision>
         </link>
         <joint name="dummy_joint" type="fixed">

File: urdf/rabbit/rabbit.urdf.xacro (robot description, xacro)
@@ -47,3 +47,11 @@
                       rpy="0.0 0.0 0.0"/>
     </xacro:if>
+    <xacro:if value="$(arg use_simulation)">
+        <gazebo>
+            <plugin name="rc_ros_control" filename="librc_robot_hw_sim.so">
+                <robotNamespace>/</robotNamespace>
+                <robotSimType>rc_gazebo/rcRobotHWSim</robotSimType>
+            </plugin>
+        </gazebo>
+    </xacro:if>
 </robot>
